Commit message: Add files via upload

File: src/maze_bot/urdf/maze_bot.urdf (robot description, URDF)
Before this commit: robot maze_bot, 6 links, 5 joints
Links:
- link base: geometry collision mesh filename=package://src/maze_bot/meshes/base_link.stl; visual mesh filename=package://src/maze_bot/meshes/base_link.stl
- link caster: geometry collision mesh filename=package://src/maze_bot/meshes/front_caster.stl; visual mesh filename=package://src/maze_bot/meshes/front_caster.stl
- link wheel_left: geometry collision mesh filename=package://src/maze_bot/meshes/wheel_l.stl; visual mesh filename=package://src/maze_bot/meshes/wheel_l.stl
- link wheel_right: geometry collision mesh filename=package://src/maze_bot/meshes/wheel_r.stl; visual mesh filename=package://src/maze_bot/meshes/wheel_r.stl
